File: cape/bela_cape_rev_C2/bela_cape.kicad_pcb (KiCad board)
At the start: 4 copper layers, 71.8 x 54.6 mm, 143 parts, among them IC1 PAM8406, IC2 TLV320AIC3104, IC3 MIC5317, IC4 TL974, IC5 TL974, IC6 ES9080Q, IC7 TSV524xIQ4T, IC8 TSV524xIQ4T, IC9 ADS8168, J1 Conn_01x02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

Commit message: Bela cape rev. C2
(cherry picked from commit 085b3700cd1d9a25c77092a8b59a7c103f45927b)
Parts:
- added R46: 100, Resistor_SMD:R_0603_1608Metric, B.Cu at (120.7, 111.0)
- added R47: 100, Resistor_SMD:R_0603_1608Metric, B.Cu at (143.7, 111.1)
- added R48: 100, Resistor_SMD:R_0603_1608Metric, B.Cu at (122.2, 111.0)
- added R49: 100, Resistor_SMD:R_0603_1608Metric, B.Cu at (145.3, 111.1)
- added R50: 100, Resistor_SMD:R_0603_1608Metric, B.Cu at (123.7, 111.0)
- added R51: 100, Resistor_SMD:R_0603_1608Metric, B.Cu at (142.1, 111.1)
- added R52: 100, Resistor_SMD:R_0603_1608Metric, B.Cu at (125.2, 111.0)
- added R53: 100, Resistor_SMD:R_0603_1608Metric, B.Cu at (140.5, 111.1)
- R1, R2: value 22k -> 51k
- moved C38 0.70 mm to (128.0, 110.2)
Connections:
- IC6 pad 22: /Analog Output/DAC7 -> Net-(IC6-Pad22)
- IC6 pad 23: /Analog Output/DAC5 -> Net-(IC6-Pad23)
- IC6 pad 24: /Analog Output/GND_SNS_R -> GNDA
- IC6 pad 25: /Analog Output/DAC3 -> Net-(IC6-Pad25)
- IC6 pad 26: /Analog Output/DAC1 -> Net-(IC6-Pad26)
- IC6 pad 5: /Analog Output/DAC0 -> Net-(IC6-Pad5)
- IC6 pad 6: /Analog Output/DAC2 -> Net-(IC6-Pad6)
- IC6 pad 7: /Analog Output/GND_SNS_L -> GNDA
- IC6 pad 8: /Analog Output/DAC4 -> Net-(IC6-Pad8)
- IC6 pad 9: /Analog Output/DAC6 -> Net-(IC6-Pad9)
Routing:
- net GNDA: track 145.8 -> 165.0 mm, vias 52 -> 53
- net Net-(IC6-Pad26): track 0.00 -> 16.7 mm, vias 0 -> 2
- net Net-(IC6-Pad25): track 0.00 -> 14.9 mm
- net Net-(IC6-Pad5): track 0.00 -> 12.3 mm, vias 0 -> 2
- net Net-(IC6-Pad6): track 0.00 -> 10.7 mm, vias 0 -> 2
- net /Analog Output/DAC3: track 42.6 -> 32.6 mm
- net Net-(IC6-Pad8): track 0.00 -> 7.82 mm
- net /Analog Output/DAC4: track 21.5 -> 13.9 mm
- net Net-(IC6-Pad23): track 0.00 -> 7.57 mm
- net /Analog Output/DAC5: track 27.3 -> 19.7 mm
- net /Analog Output/DAC6: track 20.5 -> 14.4 mm
- net /Analog Output/DAC7: track 28.3 -> 22.4 mm
- net Net-(IC6-Pad9): track 0.00 -> 5.80 mm
- net /Analog Output/DAC1: track 39.6 -> 34.1 mm
- net /Analog Output/DAC2: track 36.8 -> 31.6 mm
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Other:
- board text added: "11/22 rev. C2"
- board text removed: "10/22 rev. C1"

Commit message: A few edits to C2 cape
(cherry picked from commit 42570a0d57f5cd6d8ff56c36d77f2d0b211cc62f)
Parts:
- added R54: 4.7k, Resistor_SMD:R_0603_1608Metric, B.Cu at (174.1, 124.5)
- R46, R47, R48, R49, R50, R51, R52, R53: value 100 -> 330
- moved R36 0.41 mm to (174.1, 126.0)
Routing:
- net +3V3: track 182.0 -> 206.4 mm, vias 11 -> 12
- net GND: track 108.0 -> 104.0 mm
- net /SHUTDOWN_REQ/: track 28.4 -> 30.5 mm
