File: cape/bela_cape_rev_C3/bela_cape.kicad_pcb (KiCad board)
At the start: 4 copper layers, 71.8 x 54.6 mm, 152 parts, among them IC1 PAM8406, IC2 TLV320AIC3104, IC3 MIC5317, IC4 MC33204, IC5 MC33204, IC6 ES9080Q, IC7 TSV524xIQ4T, IC8 TSV524xIQ4T, IC9 ADS8168, J1 Conn_01x02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

Commit message: Add analog out connection to P8.15 for future BBAI64 support
Parts:
- added R55: DNI, Resistor_SMD:R_0603_1608Metric, B.Cu at (134.0, 84.1)
Connections:
- P1 pad P8.15: unconnected-(P1-PadP8.15) -> Net-(P1-PadP8.15)
Routing:
- net Net-(P1-PadP8.15): track 0.00 -> 2.01 mm
- net AUD_DOUT2: track 91.3 -> 92.2 mm
- net GND: vias 16 -> 18
Changed lines of the file:
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@@
   (net 46 "unconnected-(P1-PadP8.13)")
   (net 47 "unconnected-(P1-PadP8.14)")
-  (net 48 "unconnected-(P1-PadP8.15)")
+  (net 48 "Net-(P1-PadP8.15)")
   (net 49 "unconnected-(P1-PadP8.16)")
   (net 50 "unconnected-(P1-PadP8.18)")
@@
       (net 47 "unconnected-(P1-PadP8.14)") (pinfunction "GPIO_26") (pintype "bidirectional+no_connect"))
     (pad "P8.15" thru_hole oval (at 25.36 -8.51 90) (size 1.7272 1.7272) (drill 1.016) (layers *.Cu *.Mask "F.SilkS")
-      (net 48 "unconnected-(P1-PadP8.15)") (pinfunction "GPIO_47") (pintype "bidirectional+no_connect"))
+      (net 48 "Net-(P1-PadP8.15)") (pinfunction "GPIO_47") (pintype "bidirectional"))
     (pad "P8.16" thru_hole oval (at 27.9 -8.51 90) (size 1.7272 1.7272) (drill 1.016) (layers *.Cu *.Mask "F.SilkS")
       (net 49 "unconnected-(P1-PadP8.16)") (pinfunction "GPIO_46") (pintype "bidirectional+no_connect"))
@@
     )
   )
+  (footprint "Resistor_SMD:R_0603_1608Metric" (layer "B.Cu")
+    (at 134 84.1)
+    (descr "Resistor SMD 0603 (1608 Metric), square (rectangular) end terminal, IPC_7351 nominal, (Body size source: IPC-SM-782 page 72, https://www.pcb-3d.com/wordpress/wp-content/uploads/ipc-sm-782a_amendment_1_and_2.pdf), generated with kicad-footprint-generator")
+    (tags "resistor")
+    (property "Sheetfile" "bela_cape.kicad_sch")
+    (property "Sheetname" "")
+    (property "manf#" "ASC0603-10KFT5")
+    (attr smd)
+    (fp_text reference "R55" (at -2.8 0.1) (layer "B.SilkS")
+      (effects (font (size 0.8 0.8) (thickness 0.15)) (justify mirror))
+    )
+    (fp_text value "DNI" (at 0 -1.43) (layer "B.Fab")
+      (effects (font (size 1 1) (thickness 0.15)) (justify mirror))
+    )
+    (fp_text user "${REFERENCE}" (at 0 0) (layer "B.Fab")
+      (effects (font (size 0.4 0.4) (thickness 0.06)) (justify mirror))
+    )
+    (fp_line (start -0.237258 -0.5225) (end 0.237258 -0.5225) (layer "B.SilkS") (width 0.12))
+    (fp_line (start -0.237258 0.5225) (end 0.237258 0.5225) (layer "B.SilkS") (width 0.12))
+    (fp_line (start -1.48 -0.73) (end -1.48 0.73) (layer "B.CrtYd") (width 0.05))
+    (fp_line (start 1.48 -0.73) (end -1.48 -0.73) (layer "B.CrtYd") (width 0.05))
+    (fp_line (start -1.48 0.73) (end 1.48 0.73) (layer "B.CrtYd") (width 0.05))
+    (fp_line (start 1.48 0.73) (end 1.48 -0.73) (layer "B.CrtYd") (width 0.05))
+    (fp_line (start -0.8 0.4125) (end 0.8 0.4125) (layer "B.Fab") (width 0.1))
+    (fp_line (start 0.8 -0.4125) (end -0.8 -0.4125) (layer "B.Fab") (width 0.1))
+    (fp_line (start 0.8 0.4125) (end 0.8 -0.4125) (layer "B.Fab") (width 0.1))
+    (fp_line (start -0.8 -0.4125) (end -0.8 0.4125) (layer "B.Fab") (width 0.1))
+    (pad "1" smd roundrect (at -0.825 0) (size 0.8 0.95) (layers "B.Cu" "B.Paste" "B.Mask") (roundrect_rratio 0.25)
+      (net 99 "AUD_DOUT2") (pintype "passive"))
+    (pad "2" smd roundrect (at 0.825 0) (size 0.8 0.95) (layers "B.Cu" "B.Paste" "B.Mask") (roundrect_rratio 0.25)
+      (net 48 "Net-(P1-PadP8.15)") (pintype "passive"))
+    (model "${KICAD6_3DMODEL_DIR}/Resistor_SMD.3dshapes/R_0603_1608Metric.wrl"
+      (offset (xyz 0 0 0))
+      (scale (xyz 1 1 1))
+      (rotate (xyz 0 0 0))
+    )
+  )
   (footprint "Capacitor_SMD:C_0603_1608Metric" (layer "B.Cu")
     (at 122.85 103.2 90)
@@
   (via (at 131.5 124.9) (size 0.8) (drill 0.4) (layers "F.Cu" "B.Cu") (free) (net 6))
   (via (at 124.1 119.3) (size 0.8) (drill 0.4) (layers "F.Cu" "B.Cu") (free) (net 6))
+  (via (at 146.25 84.05) (size 0.8) (drill 0.4) (layers "F.Cu" "B.Cu") (free) (net 6))
   (via (at 126.45 116.55) (size 0.8) (drill 0.4) (layers "F.Cu" "B.Cu") (net 6))
   (via (at 123.3 125.9) (size 0.8) (drill 0.4) (layers "F.Cu" "B.Cu") (free) (net 6))
@@
   (via (at 148.554193 119.279894) (size 0.8) (drill 0.4) (layers "F.Cu" "B.Cu") (net 6))
   (via (at 121 125.9) (size 0.8) (drill 0.4) (layers "F.Cu" "B.Cu") (free) (net 6))
+  (via (at 138.6 84.05) (size 0.8) (drill 0.4) (layers "F.Cu" "B.Cu") (free) (net 6))
   (via (at 159 84.4) (size 0.8) (drill 0.4) (layers "F.Cu" "B.Cu") (free) (net 6))
   (segment (start 144.955 90.48644) (end 140.772699 94.668741) (width 0.3) (layer "In2.Cu") (net 6))
@@
   (segment (start 160.92 118.84) (end 164.26 118.84) (width 0.2) (layer "B.Cu") (net 35))
   (segment (start 164.26 118.84) (end 166.5 116.6) (width 0.2) (layer "B.Cu") (net 35))
+  (segment (start 134.825 84.2) (end 134.83 84.195) (width 0.2) (layer "B.Cu") (net 48))
+  (segment (start 134.83 84.195) (end 134.83 82.195) (width 0.2) (layer "B.Cu") (net 48))
   (segment (start 123.6375 123.9375) (end 122.13 125.445) (width 0.3) (layer "B.Cu") (net 74))
   (segment (start 122.13 125.445) (end 122.13 127.915) (width 0.3) (layer "B.Cu") (net 74))
@@
   (via (at 133.91 116.7727) (size 0.8) (drill 0.4) (layers "F.Cu" "B.Cu") (net 99))
   (via (at 129.05 117.85) (size 0.8) (drill 0.4) (layers "F.Cu" "B.Cu") (net 99))
-  (segment (start 120.95 117.85) (end 129.05 117.85) (width 0.2) (layer "B.Cu") (net 99))
-  (segment (start 156.055 84.57) (end 116.13 84.57) (width 0.2) (layer "B.Cu") (net 99))
-  (segment (start 115.306287 89.297689) (end 119.102311 93.093713) (width 0.2) (layer "B.Cu") (net 99))
+  (segment (start 120.95 117.85) (end 119.102311 116.002311) (width 0.2) (layer "B.Cu") (net 99))
+  (segment (start 129.05 117.85) (end 120.95 117.85) (width 0.2) (layer "B.Cu") (net 99))
+  (segment (start 119.102311 93.093713) (end 115.306287 89.297689) (width 0.2) (layer "B.Cu") (net 99))
+  (segment (start 119.102311 116.002311) (end 119.102311 93.093713) (width 0.2) (layer "B.Cu") (net 99))
+  (segment (start 147.3 84.2) (end 155.685 84.2) (width 0.2) (layer "B.Cu") (net 99))
+  (segment (start 133.975 84.9) (end 146.6 84.9) (width 0.2) (layer "B.Cu") (net 99))
   (segment (start 132.75 116.53) (end 132.9927 116.7727) (width 0.2) (layer "B.Cu") (net 99))
+  (segment (start 115.306287 89.297689) (end 115.306287 85.393713) (width 0.2) (layer "B.Cu") (net 99))
   (segment (start 132.9927 116.7727) (end 133.91 116.7727) (width 0.2) (layer "B.Cu") (net 99))
-  (segment (start 116.13 84.57) (end 115.306287 85.393713) (width 0.2) (layer "B.Cu") (net 99))
+  (segment (start 146.6 84.9) (end 147.3 84.2) (width 0.2) (layer "B.Cu") (net 99))
+  (segment (start 115.306287 85.393713) (end 116.5 84.2) (width 0.2) (layer "B.Cu") (net 99))
   (segment (start 132.75 115.8) (end 132.75 116.53) (width 0.2) (layer "B.Cu") (net 99))
-  (segment (start 115.306287 85.393713) (end 115.306287 89.297689) (width 0.2) (layer "B.Cu") (net 99))
-  (segment (start 119.102311 93.093713) (end 119.102311 116.002311) (width 0.2) (layer "B.Cu") (net 99))
-  (segment (start 119.102311 116.002311) (end 120.95 117.85) (width 0.2) (layer "B.Cu") (net 99))
+  (segment (start 155.685 84.2) (end 156.055 84.57) (width 0.2) (layer "B.Cu") (net 99))
+  (segment (start 133.275 84.2) (end 133.975 84.9) (width 0.2) (layer "B.Cu") (net 99))
+  (segment (start 116.5 84.2) (end 133.275 84.2) (width 0.2) (layer "B.Cu") (net 99))
   (segment (start 139.9 89.075) (end 139.9 87.25) (width 0.2) (layer "B.Cu") (net 100))
   (segment (start 137.35 89.125) (end 137.35 87.26) (width 0.2) (layer "B.Cu") (net 101))

Commit message: removed sym-lib-table with a reference to an unused and obsolete local library
Other:
- board text added: "02/23 rev. ${REVISION}"
- board text removed: "02/23 rev. C3"
