File: cape/bela_cape_rev_C3/bela_cape.kicad_sch (KiCad schematic)
At the start: 35 parts, among them J1 Conn_01x02, J10 Conn_01x04, J11 Conn_01x02, J2 Conn_01x04, J3 Conn_01x03, J4 Conn_01x03, J5 Conn_01x02, J6 Conn_01x02, J7 Conn_01x10, J8 Conn_01x10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

Commit message: Add analog out connection to P8.15 for future BBAI64 support
Parts:
- added R55: DNI, Resistor_SMD:R_0603_1608Metric, symbol Device:R
Connections:
- net AUD_DOUT2: now also R55.1
- net at P1.P8.15 (GPIO_47): now also R55.2
- no-connect marks 58 -> 57
Changed lines of the file:
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@@
   (no_connect (at 203.2 33.02))
   (no_connect (at 203.2 81.28))
-  (no_connect (at 203.2 48.26))
   (no_connect (at 203.2 35.56))
   (no_connect (at 236.22 116.84))
@@
     (stroke (width 0) (type default) (color 0 0 0 0))
   )
+  (wire (pts (xy 193.04 48.26) (xy 194.31 48.26))
+    (stroke (width 0) (type default) (color 0 0 0 0))
+  )
   (wire (pts (xy 104.14 93.98) (xy 111.76 93.98))
     (stroke (width 0) (type default) (color 0 0 0 0))
@@
   )
   (wire (pts (xy 111.76 46.99) (xy 113.03 45.72))
+    (stroke (width 0) (type default) (color 0 0 0 0))
+  )
+  (wire (pts (xy 201.93 48.26) (xy 203.2 48.26))
     (stroke (width 0) (type default) (color 0 0 0 0))
   )
@@
     )
   )
+  (global_label "AUD_DOUT2" (shape input) (at 193.04 48.26 180) (fields_autoplaced)
+    (effects (font (size 1.27 1.27)) (justify right))
+    (property "Intersheet References" "${INTERSHEET_REFS}" (id 0) (at 179.8621 48.1806 0)
+      (effects (font (size 1.27 1.27)) (justify right) hide)
+    )
+  )
   (global_label "RESETN" (shape input) (at 247.65 111.76 0) (fields_autoplaced)
     (effects (font (size 1.27 1.27)) (justify left))
@@
     )
     (pin "1")
+  )
+  (symbol (lib_id "Device:R") (at 198.12 48.26 90) (unit 1)
+    (in_bom yes) (on_board yes)
+    (property "Reference" "R55" (id 0) (at 198.12 50.8 90))
+    (property "Value" "DNI" (id 1) (at 198.12 53.34 90))
+    (property "Footprint" "Resistor_SMD:R_0603_1608Metric" (id 2) (at 198.12 50.038 90)
+      (effects (font (size 1.27 1.27)) hide)
+    )
+    (property "Datasheet" "~" (id 3) (at 198.12 48.26 0)
+      (effects (font (size 1.27 1.27)) hide)
+    )
+    (property "manf#" "ASC0603-10KFT5" (id 4) (at 198.12 48.26 0)
+      (effects (font (size 1.27 1.27)) hide)
+    )
+    (pin "1")
+    (pin "2")
   )
   (symbol (lib_id "power:GNDA") (at 101.6 140.97 0) (unit 1)
@@
       (reference "R54") (unit 1) (value "4.7k") (footprint "Resistor_SMD:R_0603_1608Metric")
     )
+    (path "/2f00568c-bea1-43f5-930d-5b8197e322b2"
+      (reference "R55") (unit 1) (value "DNI") (footprint "Resistor_SMD:R_0603_1608Metric")
+    )
     (path "/63b54547-a58e-47a7-8ea4-655fb9be79b4"
