File: GemMulti/GemMulti_rev_A4/bela_mini_multi_pb2.kicad_pcb (KiCad board)
At the start: 4 copper layers, 55 x 66 mm, 35 parts, among them J1 AudioJack4, J10 Conn_01x03, J11 Conn_01x03, J12 Conn_01x02, J2 AudioJack4, J3 Conn_01x10, J4 Conn_01x04_MountingPin, J5 USB_A, J6 Conn_02x12_Odd_Even, J7 Conn_02x11_Odd_Even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

Commit message: removed logos
Parts:
- removed G***: LOGO, LOGO
