File: GemStereo/GemStereo_rev_A4/bela_mini_pb2_square.kicad_pcb (KiCad board)
At the start: 4 copper layers, 55 x 44.6 mm, 28 parts, among them J1 Conn_01x03, J2 Conn_01x03, J3 Conn_01x10, J5 USB_A, J6 Conn_01x04_MountingPin, J7 AudioJack4, J8 AudioJack4, J9 Conn_01x05, U1 PocketBeagle2

Commit message: removed logos
Parts:
- removed G***: LOGO, LOGO
